File: ChessBotController.kicad_pcb (KiCad board)
At the start: 4 copper layers, 71.3 x 95.9 mm, 51 parts, among them J1 PART_FAN, J10 Z_END, J11 PWR_ALT, J2 PWR_ATX, J3 HEATBED, J4 HOTEND, J5 BED, J6 HOTEND, J7 HEATBRK_FAN, J8 LCD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

Commit message: feat: initial v0.2 design
Parts:
- removed R1, R3: 1k, Resistor_THT:R_Axial_DIN0207_L6.3mm_D2.5mm_P7.62mm_Horizontal
- added JP1: USB_PWR, Connector_PinHeader_2.54mm:PinHeader_1x02_P2.54mm_Vertical, F.Cu at (138.9, 119.5)
- added R10: 1k, Resistor_THT:R_Axial_DIN0207_L6.3mm_D2.5mm_P7.62mm_Horizontal, F.Cu at (133.1, 76.7)
- added R9: 1k, Resistor_THT:R_Axial_DIN0207_L6.3mm_D2.5mm_P7.62mm_Horizontal, F.Cu at (143.0, 76.7)
- added SW1: SW_Push, Button_Switch_THT:SW_PUSH_6mm, F.Cu at (128.5, 60.6)
- added SW2: SW_Push, Button_Switch_THT:SW_PUSH_6mm, F.Cu at (146.8, 115.2)
- added U10: ESP32-WROOM-E, Espressif:ESP32-WROOM-32E, F.Cu at (140.6, 63.1)
- U3: value ESP32 DevKit -> Adafruit-CH2102N-Friend; footprint Espressif:ESP32-DevKitC -> USB_to_Serial_Friend:Adafruit-CH2102N-Friend
- moved J11 82.8 mm to (122.0, 147.6), turned to 0 degrees
- moved REF** 40.7 mm to (186.1, 53.8)
- moved C7 40.5 mm to (134.4, 113.4), turned to 180 degrees
- moved U3 33.1 mm to (152.9, 121.4), turned to -90 degrees
- moved J9 32.3 mm to (124.9, 111.3)
- moved C8 29.7 mm to (133.5, 122.3)
- moved J10 26.0 mm to (124.9, 107.4)
- moved U8 24.8 mm to (150.7, 99.3), turned to 180 degrees
- moved J4 19.4 mm to (124.9, 78.5)
- moved U9 18.1 mm to (132.3, 81.5), turned to 0 degrees
- moved J8 13.4 mm to (124.9, 92.6)
- moved J7 12.8 mm to (130.6, 138.9), turned to 90 degrees
- moved R7 10.1 mm to (124.9, 127.4), turned to 90 degrees
- moved R2 10.1 mm to (124.9, 132.0), turned to -90 degrees
- moved J5 6.84 mm to (124.9, 84.8)
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Connections:
- net Net-(J2-+3.3V-Pad1) renamed +3.3VP
- U3 pad 1: +3V3 -> GND
- U3 pad 10: /SDA -> +3V3
- U3 pad 11: /HOTEND_H -> GND
- U3 pad 12: /FAN_0 -> unconnected-(U3-RST-Pad12)
- U3 pad 14: GND -> unconnected-(U3-IO2-Pad14)
- U3 pad 15: Net-(U3-MTCK/GPIO13/ADC2_CH4) -> unconnected-(U3-SU#-Pad15)
- U3 pad 17: unconnected-(U3-SD_DATA3/GPIO10-Pad17) -> unconnected-(U3-CTS-Pad17)
- U3 pad 18: unconnected-(U3-CMD-Pad18) -> Net-(U3-RTS-Pad18)
- U3 pad 19: +5V -> /MCU_TXD
- U3 pad 2: unconnected-(U3-CHIP_PU-Pad2) -> unconnected-(U3-CTS-Pad17)
- U3 pad 20: unconnected-(U3-SD_CLK/GPIO6-Pad20) -> /MCU_RXD
- U3 pad 3: /TEMP_HOTEND -> Net-(JP1-B)
- U3 pad 4: /TEMP_BED -> /MCU_TXD
- U3 pad 5: /Y_MIN -> /MCU_RXD
- U3 pad 8: /BED_H -> Net-(U3-RTS-Pad18)
- U3 pad 9: /SCL -> Net-(JP1-B)
- U5 pad 5: /DRIVER_UART_1 -> /DRIVER_UART_2
- U7 pad 5: /DRIVER_UART_2 -> /DRIVER_UART_1
- U8 pad 1: /Y_DIR -> /X_STEP
- U8 pad 2: /Y_STEP -> /X_DIR
- U8 pad 3: /X_STEP -> /Y_DIR
- U8 pad 4: /X_DIR -> /Y_STEP
Routing:
- net /MCU_RXD: track 0.00 -> 85.6 mm, vias 0 -> 1
- net /MCU_TXD: track 0.00 -> 79.9 mm, vias 0 -> 1
- net /Z_MIN: track 8.72 -> 72.3 mm, vias 0 -> 1
- net /FAN_0: track 19.1 -> 72.8 mm
- net /BED_H: track 9.71 -> 61.0 mm
- net /HOTEND_H: track 16.0 -> 65.7 mm
- net Net-(U10-GPIO0/BOOT/ADC2_CH1): track 0.00 -> 43.6 mm, vias 0 -> 1
- net /TEMP_HOTEND: track 10.2 -> 48.9 mm
- net /DRIVER_UART_2: track 69.8 -> 100.6 mm, vias 0 -> 1
- net /TEMP_BED: track 20.1 -> 50.7 mm
- net Net-(JP1-B): track 0.00 -> 28.8 mm
- net /Y_MIN: track 58.7 -> 32.1 mm, vias 0 -> 1
- net /X_DIR: track 46.5 -> 23.4 mm
- net /X_STEP: track 39.8 -> 19.8 mm
- net /DRIVER_UART_1: track 89.8 -> 73.4 mm, vias 0 -> 1
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Other:
- board text added: "v0.2"
- board text removed: "A chess bot, but on steroids"
- board text removed: "v0.1"
