File: ChessBotController.kicad_sch (KiCad schematic)
At the start: 14 parts, among them J8 LCD, U3 ESP32 DevKit, U8 74HC595, U9 74HC595

Commit message: feat: initial v0.2 design
Parts:
- removed R1, R3: 1k, Resistor_THT:R_Axial_DIN0207_L6.3mm_D2.5mm_P7.62mm_Horizontal, symbol Device:R
- removed U3: ESP32 DevKit, Espressif:ESP32-DevKitC, symbol Espressif:ESP32-DevKitC
- added JP2: USB_PWR, Connector_PinHeader_2.54mm:PinHeader_1x02_P2.54mm_Vertical, symbol Jumper:Jumper_2_Bridged
- added R10, R9: 1k, Resistor_THT:R_Axial_DIN0207_L6.3mm_D2.5mm_P7.62mm_Horizontal, symbol Device:R
- added SW1, SW2: SW_Push, Button_Switch_THT:SW_PUSH_6mm, symbol Switch:SW_Push
- added U10: ESP32-WROOM-E, Espressif:ESP32-WROOM-32E, symbol Espressif:ESP32-WROOM-E
- added U3: Adafruit-CH2102N-Friend, USB_to_Serial_Friend:Adafruit-CH2102N-Friend, symbol USB_to_Serial:Adafruit-CH2102N-Friend
Connections:
- net +3V3: now also U10.2 (3V3), U3.10 (3V3)
- net +5V: now also JP2.1 (A)
- net BED_H: now also U10.9 (32K_XN/GPIO33/ADC1_CH5)
- net DRIVER_UART_1: now also R9.2, U10.27 (GPIO16)
- net DRIVER_UART_2: now also R10.2, U10.26 (ADC2_CH0/GPIO4)
- net FAN_0: now also U10.13 (MTMS/GPIO14/ADC2_CH6)
- net GND: now also SW1.1, SW2.2, U10.1 (GND), U10.15 (GND), U10.38 (GND), U10.39 (GND_THERMAL), U3.1 (GND), U3.11 (GND)
- net HOTEND_H: now also U10.12 (ADC2_CH7/GPIO27)
- net I2S_BCK: now also U10.36 (GPIO22)
- net I2S_DIN: now also U10.31 (GPIO19)
- net I2S_WCK: now also U10.33 (GPIO21)
- net PS_ON: now also U10.8 (32K_XP/GPIO32/ADC1_CH4)
- net SCL: now also U10.10 (DAC_1/ADC2_CH8/GPIO25)
- net SDA: now also U10.11 (DAC_2/ADC2_CH9/GPIO26)
- net SERVO: now also U10.30 (GPIO18)
- net TEMP_BED: now also U10.5 (SENSOR_VN/GPIO39/ADC1_CH3)
- net TEMP_HOTEND: now also U10.4 (SENSOR_VP/GPIO36/ADC1_CH0)
- net X_DIR: now also U8.2 (QC); no longer U8.4 (QE)
- net X_MIN: now also U10.7 (GPIO35/ADC1_CH7)
- net X_STEP: now also U8.1 (QB); no longer U8.3 (QD)
- net Y_DIR: now also U8.3 (QD); no longer U8.1 (QB)
- net Y_MIN: now also U10.6 (GPIO34/ADC1_CH6)
- net Y_STEP: now also U8.4 (QE); no longer U8.2 (QC)
- net Z_MIN: now also U10.37 (GPIO23)
- new net: SW2.1, U10.25 (GPIO0/BOOT/ADC2_CH1)
- new net: SW1.2, U10.3 (EN/CHIP_PU)
- new net: R10.1, U10.16 (MTCK/GPIO13/ADC2_CH4)
- new net: R9.1, U10.28 (GPIO17)
- new net: JP2.2 (B), U3.3 (5V), U3.9 (5V)
- new net: U3.17 (CTS), U3.2 (CTS)
- new net: U3.18 (RTS), U3.8 (RTS)
- new net MCU_RXD: U10.34 (U0RXD/GPIO3), U3.20 (TXD), U3.5 (TXD)
- new net MCU_TXD: U10.35 (U0TXD/GPIO1), U3.19 (RXD), U3.4 (RXD)
Other:
- moved on the sheet: J8
