File: pwr.kicad_sch (KiCad schematic)
At the start: 3 parts, among them J11 PWR_ALT, J2 PWR_ATX

Commit message: feat: initial v0.2 design
Connections:
- net +3.3VP: now reaches J2.1 (+3.3V), J2.12 (+3.3V), J2.13 (+3.3V), J2.2 (+3.3V)
- no-connect marks 0 -> 1
Other:
- moved on the sheet: J11, J2, JP2
